File: SD_CARD.kicad_pcb (KiCad board)
At the start: 2 copper layers, 33.5 x 25 mm, 12 parts, among them P1 CONN_01X07

Commit message: added corrected files
Parts:
- added LOGO: , LOGO:LOGO (2), B.Cu at (49.0, 32.5)
- D1, D2, D3: footprint Diodes_SMD:Diode-SMA_Handsoldering -> ee:ZenerDiode_SMD
- moved C1 86.4 mm to (43.7, 34.8)
- moved C2 86.4 mm to (41.2, 34.8)
- moved D1 86.4 mm to (56.2, 41.4), turned to 0 degrees
- moved D2 86.4 mm to (56.2, 37.6), turned to 0 degrees
- moved D3 86.4 mm to (56.2, 33.8), turned to 0 degrees
- moved P1 86.4 mm to (65.6, 44.9)
- moved R1 86.4 mm to (43.2, 41.6)
- moved R2 86.4 mm to (54.9, 44.7)
- moved R3 86.4 mm to (54.9, 27.9)
- moved R4 86.4 mm to (54.9, 30.5)
- moved SD1 86.4 mm to (48.3, 35.0)
- moved R5 86.4 mm to (54.9, 47.2)
Routing:
- net /SD_DETECT: track 41.7 -> 44.8 mm
- added copper zone on F.Cu, net 5V
- added copper zone on B.Cu, net GND
Other:
- outline, holes or cut-outs redrawn
- board text added: "COMP"
- board text added: "ExploreEmbedded.com"
- board text added: "SOLD"
